Commit message: URDF with link tags mostly complete remember to finish off joints and add an actuator tag

File: urdf/rover_arm.urdf (robot description, URDF)
Before this commit: robot rover_arm, 4 links, 0 joints
Links:
- link Elbow: mass None -> 0.602; geometry visual cylinder length=0.21 radius=0.03
- link Shoulder: mass None -> 2.333; geometry visual cylinder length=0.41 radius=0.04
- link Wrist: mass None -> 2.128; geometry collision box size=0.33 0.1 0.06; visual box size=0.33 0.1 0.06
- link base: mass None -> 1.206; geometry collision box size=.13 0.13 0.11; visual box size=0.13 0.13 0.11

Commit message: URDF with link tags mostly complete save the actuator/transmission tage for the shoulder. Also made the joints need to test out what the positions actually look like later

File: urdf/rover_arm.urdf (robot description, URDF)
Before this commit: robot rover_arm, 4 links, 0 joints
Links:
- added link elbow_to_wrist_continuous
- added link virtual_base_to_shoulder
- added link world
- link Elbow: geometry visual origin rpy=0.0 0.0 0.0 xyz=0.1 0.41 0.0
- link Shoulder: geometry visual origin rpy=0.0 0.0 1.5707 xyz=0.0 0.0 0.0
- link Wrist: geometry collision origin rpy=0.0 0.0 0.0 xyz=0.21 0.41 0.0; visual origin rpy=0.0 0.0 0.0 xyz=0.21 0.41 0.0
Joints:
- added joint base_to_shoulder_rotatexy: type revolute, parent base, child shoulder, origin xyz=0.0 0.0 0.0 rpy=0.0 0.0 0.0, axis 0.0 0.0 1.0, limit lower=0.0 upper=6.28 effort=10.0 velocity=10.0
- added joint base_to_shoulder_rotatezx: type revolute, parent base, child shoulder, origin xyz=0.0 0.0 0.0 rpy=0.0 0.0 0.0, axis 0.0 1.0 0.0, limit lower=0.5 upper=1.5707 effort=10.0 velocity=10.0
- added joint elbow_to_wrist_cont: type continuous, parent elbow, child wrist, origin xyz=0.0 0.0 0.0 rpy=0.0 0.0 0.0, axis 0.0 1.0 0.0
- added joint elbow_to_wrist_revolve: type revolute, parent elbow, child wrist, origin xyz=0.0 0.0 0.0 rpy=0.0 0.0 0.0, axis 1.0 0.0 0.0, limit lower=-1.5707 upper=1.5707 effort=10.0 velocity=10.0
- added joint shoulder_to_elbow: type revolute, parent shoulder, child elbow, origin xyz=0.0 0.0 0.0 rpy=0.0 0.0 0.0, axis 0.0 1.0 0.0, limit lower=0.5 upper=1.5707 effort=10.0 velocity=10.0
- added joint world_to_base: type fixed, parent world, child base, origin xyz=0.0 0.0 0.0 rpy=0.0 0.0 0.0

Commit message: Fixed most syntax errors on the file, remaining error is that gazebo cannot resolve the virtual joint and the actual

File: urdf/rover_arm.urdf (robot description, URDF)
Before this commit: robot rover_arm, 7 links, 6 joints
Links:
- removed link Elbow
- removed link Shoulder
- removed link Wrist
- added link elbow, mass 0.602; collision cylinder length=0.21 radius=0.03; visual cylinder length=0.21 radius=0.03
- added link shoulder, mass 2.333; collision cylinder length=0.41 radius=0.04; visual cylinder length=0.41 radius=0.04
- added link wrist, mass 2.128; collision box size=0.33 0.1 0.06; visual box size=0.33 0.1 0.06
- link elbow_to_wrist_continuous: mass None -> 0.025
- link virtual_base_to_shoulder: mass None -> 0.025

Commit message: Added mimic tags to each of the joints where 2 DOF are needed, still need to experiment with them though, I'm unsure what the multiplier or offset buttons even do

File: urdf/rover_arm.urdf (robot description, URDF)
Before this commit: robot rover_arm, 7 links, 6 joints
Joints:
- joint base_to_shoulder_rotatezx: mimic (none) -> joint=base_to_shoulder_rotatexy
- joint elbow_to_wrist_cont: mimic (none) -> joint=elbow_to_wrist_revolve
